Commit message: model updates

File: p3at_description/urdf/pioneer3at.urdf.xacro (robot description, xacro)
@@ -8,9 +8,4 @@
   <include filename="$(find p3at_description)/urdf/pioneer3at_body.xacro"/>
   <include filename="$(find p3at_description)/urdf/hokuyo_utm30lx.urdf.xacro"/>
-  <xacro:p3at_front suffix="left" reflect="1"/>
-  <xacro:p3at_front suffix="right" reflect="-1"/>
-  <xacro:p3at_back suffix="left" reflect="1"/>
-  <xacro:p3at_back suffix="right" reflect="-1"/>
-  <xacro:p3at_gazebo_ext/>
   <xacro:hokuyo_utm30lx name="hokuyo" parent="base_link" ros_topic="hokuyo" update_rate="30" ray_count="1040" min_angle="130" max_angle="-130" >
     <origin xyz="0.13 0 0.32" rpy="0 0 0"/>

File: p3at_description/urdf/pioneer3at_body.xacro (robot description, xacro)
@@ -15,5 +15,5 @@
     </inertial>
     <visual name="base_visual">
-      <origin xyz="0 0 0.177" rpy="0 0 0"/>
+      <origin xyz="0 0 0.18" rpy="0 0 0"/>
       <geometry name="pioneer_geom">
         <mesh filename="package://p3at_description/meshes/p3at_meshes/chassis.dae"/>
@@ -21,15 +21,11 @@
     </visual>
     <collision>
-      <origin xyz="0 0 0.177" rpy="0 0 0"/>
+      <origin xyz="0 0 0.18" rpy="0 0 0"/>
       <geometry>
-        <box>
-          <size xyz="0.501 0.3 0.19"/>
-        </box>
+        <box size="0.501 0.3 0.19"/>
       </geometry>
     </collision>
   </link>
-<!-- Front Axles + Wheels + Hubcaps -->
-<xacro:macro name="p3at_front" params="suffix reflect">
-  <link name="p3at_front_${suffix}_wheel">
+  <link name="p3at_front_left_wheel">
     <inertial>
       <mass value="1.5"/>
@@ -45,5 +41,5 @@
     </visual>
     <collision>
-      <origin xyz="0 0 0" rpy="${-3.1415927/2} 0 0"/>
+      <origin xyz="0 0 0" rpy="0 0 0"/>
       <geometry>
         <cylinder radius="0.110" length="0.075"/>
@@ -51,26 +47,13 @@
     </collision>
   </link>
-  <joint name="p3at_front_${suffix}_wheel_joint" type="continuous">
-    <axis xyz="0 1 0"/>
-    <anchor xyz="0 0 0"/>
+  <joint name="p3at_front_left_wheel_joint" type="continuous">
+    <axis xyz="0 0 1"/>
     <limit effort="100" velocity="100" />
     <joint_properties damping="0.7"/>
-    <origin xyz="0 0 0" rpy="0 0 0"/>
-    <parent link="p3at_front_${suffix}_hub"/>
-    <child link="p3at_front_${suffix}_wheel"/>
+    <origin xyz="0.125 0.2010 0.11" rpy="1.5707 0 0"/>
+    <parent link="base_link"/>
+    <child link="p3at_front_left_wheel"/>
   </joint>
-  <gazebo reference="p3at_front_${suffix}_wheel">
-    <kp>1000000.0</kp> <!-- kp and kd for rubber -->
-    <kd>100.0</kd>
-    <mu1>10.0</mu1>
-    <mu2>1.0</mu2>
-    <fdir1>0 1 0</fdir1> <!-- is this correct? -->
-    <maxVel>1.0</maxVel>
-    <minDepth>0.00</minDepth>
-  </gazebo>
-</xacro:macro>
-<!-- Back Axles + Wheels + Hubcaps -->
-<xacro:macro name="p3at_back" params="suffix reflect">
-  <link name="p3at_back_${suffix}_wheel">
+  <link name="p3at_front_right_wheel">
     <inertial>
       <mass value="1.5"/>
@@ -86,5 +69,5 @@
     </visual>
     <collision>
-      <origin xyz="0 0 0" rpy="${-3.1415927/2} 0 0"/>
+      <origin xyz="0 0 0" rpy="0 0 0"/>
       <geometry>
         <cylinder radius="0.110" length="0.075"/>
@@ -92,23 +75,68 @@
     </collision>
   </link>
-  <joint name="p3at_back_${suffix}_wheel_joint" type="continuous">
-    <axis xyz="0 1 0"/>
-    <anchor xyz="0 0 0"/>
+  <joint name="p3at_front_right_wheel_joint" type="continuous">
+    <axis xyz="0 0 1"/>
     <limit effort="100" velocity="100" />
     <joint_properties damping="0.7"/>
-    <origin xyz="0 0 0" rpy="0 0 0"/>
-    <parent link="p3at_back_${suffix}_hub"/>
-    <child link="p3at_back_${suffix}_wheel"/>
+    <origin xyz="0.125 -0.2010 0.11" rpy="1.5707 0 0"/>
+    <parent link="base_link"/>
+    <child link="p3at_front_right_wheel"/>
   </joint>
-  <gazebo reference="p3at_back_${suffix}_wheel">
-    <kp>1000000.0</kp> <!-- kp and kd for rubber -->
-    <kd>100.0</kd>
-    <mu1>10.0</mu1>
-    <mu2>1.0</mu2>
-    <fdir1>0 1 0</fdir1> <!-- is this correct? -->
-    <maxVel>1.0</maxVel>
-    <minDepth>0.00</minDepth>
-  </gazebo>
-</xacro:macro>
+  <link name="p3at_rear_left_wheel">
+    <inertial>
+      <mass value="1.5"/>
+      <origin xyz="0 0 0"/>
+      <inertia ixx="0.005240625" ixy="0" ixz="0"
+        iyy="0.005240625" iyz="0" izz="0.009075"/>
+    </inertial>
+    <visual name="visual">
+      <origin xyz="0 0 0" rpy="0 0 0"/>
+      <geometry name="geom">
+        <mesh filename="package://p3at_description/meshes/p3at_meshes/wheel.dae"/>
+      </geometry>
+    </visual>
+    <collision>
+      <origin xyz="0 0 0" rpy="0 0 0"/>
+      <geometry>
+        <cylinder radius="0.110" length="0.075"/>
+      </geometry>
+    </collision>
+  </link>
+  <joint name="p3at_rear_left_wheel_joint" type="continuous">
+    <axis xyz="0 0 1"/>
+    <limit effort="100" velocity="100" />
+    <joint_properties damping="0.7"/>
+    <origin xyz="-0.125 0.2010 0.11" rpy="1.5707 0 0"/>
+    <parent link="base_link"/>
+    <child link="p3at_rear_left_wheel"/>
+  </joint>
+  <link name="p3at_rear_right_wheel">
+    <inertial>
+      <mass value="1.5"/>
+      <origin xyz="0 0 0"/>
+      <inertia ixx="0.005240625" ixy="0" ixz="0"
+        iyy="0.005240625" iyz="0" izz="0.009075"/>
+    </inertial>
+    <visual name="visual">
+      <origin xyz="0 0 0" rpy="0 0 0"/>
+      <geometry name="geom">
+        <mesh filename="package://p3at_description/meshes/p3at_meshes/wheel.dae"/>
+      </geometry>
+    </visual>
+    <collision>
+      <origin xyz="0 0 0" rpy="0 0 0"/>
+      <geometry>
+        <cylinder radius="0.110" length="0.075"/>
+      </geometry>
+    </collision>
+  </link>
+  <joint name="p3at_rear_right_wheel_joint" type="continuous">
+    <axis xyz="0 0 1"/>
+    <limit effort="100" velocity="100" />
+    <joint_properties damping="0.7"/>
+    <origin xyz="-0.125 -0.2010 0.11" rpy="1.5707 0 0"/>
+    <parent link="base_link"/>
+    <child link="p3at_rear_right_wheel"/>
+  </joint>
 <xacro:macro name="p3at_gazebo_ext">
   <gazebo>
